File: kicon19-badge.kicad_pcb (KiCad board)
At the start: 2 copper layers, 61 parts, among them J1 LogicProbes, J2 Ports, J6 Conn_ARM_JTAG_SWD_20, J7 USB_B_Micro, SW1 BTN1, SW2 BTN2, SW3 BTN3, SW4 BTN4, SW5 Reset, SW6 Erase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

Commit message: WIP
Parts:
- J1, REF**: moved to B.Cu
- J2: footprint Connector_PinHeader_2.54mm:PinHeader_2x07_P2.54mm_Vertical -> Connector_PinHeader_2.54mm:PinHeader_2x07_P2.54mm_Horizontal
- J6: value Conn_ARM_JTAG_SWD_20 -> Conn_ARM_JTAG_SWD_10; footprint Connector_IDC:IDC-Header_2x10_P2.54mm_Vertical -> Connector_PinHeader_1.27mm:PinHeader_2x05_P1.27mm_Horizontal
- moved C17 220.5 mm to (435.7, 9.97)
- moved C2 220.5 mm to (376.8, 90.7)
- moved C20 220.5 mm to (326.2, 30.2)
- moved D1 220.5 mm to (385.2, 125.3)
- moved R12 220.5 mm to (455.3, 76.3)
- moved R2 220.5 mm to (396.4, 96.5)
- moved R7 220.5 mm to (446.9, 38.8)
- moved C1 220.5 mm to (379.6, 70.5)
- moved C11 220.5 mm to (427.3, 12.9)
- moved C12 220.5 mm to (430.1, 53.2)
- moved C13 220.5 mm to (402.0, 33.0)
- moved C14 220.5 mm to (382.8, 4.20)
- moved C19 220.5 mm to (410.4, 67.6)
- moved C21 220.5 mm to (390.8, 27.3)
- moved C22 220.5 mm to (421.7, 21.5)
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Connections:
- J6 pad 10: GND -> /NRST
- J6 pad 2: (no net) -> /TMS
- J6 pad 3: /NRST -> GND
- J6 pad 4: GND -> /TCK
- J6 pad 5: /TDI -> GND
- J6 pad 6: GND -> /TDO
- J6 pad 7: /TMS -> Net-(J6-Pad7)
- J6 pad 8: GND -> /TDI
- J6 pad 9: /TCK -> GND
- J7 pad 4: (no net) -> Net-(J7-Pad4)
- U3 pad 10: (no net) -> Net-(U3-Pad10)
- U3 pad 11: (no net) -> Net-(U3-Pad11)
- U3 pad 13: (no net) -> Net-(U3-Pad13)
- U3 pad 19: (no net) -> Net-(U3-Pad19)
- U3 pad 20: (no net) -> Net-(U3-Pad20)
- U3 pad 28: (no net) -> Net-(U3-Pad28)
- U3 pad 35: (no net) -> Net-(U3-Pad35)
- U3 pad 40: (no net) -> Net-(U3-Pad40)
- U3 pad 44: (no net) -> Net-(U3-Pad44)
- U3 pad 5: (no net) -> Net-(U3-Pad5)
- U3 pad 50: (no net) -> Net-(U3-Pad50)
- U3 pad 6: (no net) -> Net-(U3-Pad6)
- U3 pad 9: (no net) -> Net-(U3-Pad9)
Other:
- board outline added: 38 x 52.5 mm
- copper layers 2 -> 4
- net class Default: clearance 0.2 -> 0.15; trace_width 0.25 -> 0.15; via_dia 0.8 -> 0.6; via_drill 0.4 -> 0.3
- rule pad_to_mask_clearance: 0.051 -> 0.05
- rule solder_mask_min_width: 0.25 -> 0.05
- rule trace_clearance: 0.2 -> 0.15
- rule trace_min: 0.2 -> 0.1
- rule via_min_drill: 0.3 -> 0.2
- rule via_min_size: 0.4 -> 0.5
